Commit message: Final Visualsation and basic xml file for manipulator in mujoco( mcjf format) with all the stl files for the parts

File: urdf/manipulator_v2.urdf (robot description, URDF)
Before this commit: robot origins, 7 links, 6 joints
Links:
- link base_link: geometry collision box size=0.065 0.055 0.045; visual mesh filename=stl/umirobot_l1_meshlab.stl scale=0.01 0.01 0.01
- link l1_cover: mass 0.2 -> 0.02; geometry collision box size=0.065 0.055 0.010; visual mesh filename=stl/umirobot_l1_cover.stl scale=0.01 0.01 0.01
- link l2: mass 0.2 -> 0.08; geometry collision box size=0.065 0.035 0.055; visual mesh filename=stl/umirobot_l2_shifted.stl scale=0.01 0.01 0.01
- link l2_cover: mass 0.2 -> 0.02; geometry collision box size=0.065 0.0095 0.055; visual mesh filename=stl/umirobot_l2_cover.stl scale=0.01 0.01 0.01
- link l3: mass 0.2 -> 0.04; geometry collision box size=0.040 0.010 0.120; visual mesh filename=stl/umirobot_l3.stl scale=0.01 0.01 0.01
- link l4: mass 0.2 -> 0.05; geometry collision box size=0.120 0.025 0.040; visual mesh filename=stl/umirobot_l4.stl scale=0.01 0.01 0.01
- link l5: mass 0.2 -> 0.02; geometry collision box size=0.060 0.040 0.032; visual mesh filename=stl/umirobot_l5.stl scale=0.01 0.01 0.01
Joints:
- joint joint_l2_l3: limit lower=2.3562 upper=4.71239 effort=10.0 velocity=1.0 -> lower=-1.1781 upper=1.1781 effort=10.0 velocity=1.0
- joint joint_l3_l4: origin xyz=0 -0.4 -0.8 rpy=3.14159 0 3.14159 -> xyz=0.0 0.0 0.0 rpy=0.0 0.0 0.0
- joint joint_l4_l5: limit lower=1 upper=10 effort=10.0 velocity=1.0 -> lower=-3.14159 upper=3.14159 effort=10.0 velocity=1.0; origin xyz=1.5 0.115 -0.01 rpy=3.14159 0 3.14159 -> xyz=0.0 0.0 0.0 rpy=0.0 0.0 0.0
